File: kivy/sap-pcb.sch (KiCad schematic (older format))
At the start: 11 parts, among them P7 TE_RELAY_(ORWH-SH-112D), Q1 Q_NPN_EBC, Q10 Q_NPN, U1 Arduino_Nano

Commit message: finished circuit design.  still need to give look over.
Parts:
- removed D1: D, Diodes_ThroughHole:Diode_DO-41_SOD81_Horizontal_RM10, symbol D
- removed OUTPUTS_2, PWR_IN_1: CONN_01X04, USBdio-PCB:PHX_HDR_4_POS_(1933202), symbol CONN_01X04
- removed P7: TE_RELAY_(ORWH-SH-112D), USBdio-PCB:TE_RELAY_(ORWH-SH-112D), symbol TE_RELAY_(ORWH-SH-112D)
- removed Q1: Q_NPN_EBC, TO_SOT_Packages_THT:TO-92_Molded_Narrow, symbol Q_NPN_EBC
- removed Q10: Q_NPN, TO_SOT_Packages_THT:TO-92_Molded_Narrow, symbol Q_NPN_EBC
- removed R1, R2: 10k, Resistors_ThroughHole:Resistor_Horizontal_RM10mm, symbol R
- removed R19: 1k, Resistors_ThroughHole:Resistor_Horizontal_RM10mm, symbol R
- added CONTROL: CONN_01X15, symbol CONN_01X15
- added D?: D, symbol D
- added D? (x3): D, Diodes_ThroughHole:Diode_DO-41_SOD81_Horizontal_RM10, symbol D
- added P?: DROK_DC_DC_CONVERTOR, symbol DROK_DC_DC_CONVERTOR
- added POWER: CONN_01X03, symbol CONN_01X03
- added Q?: Q_NPN_EBC, TO_SOT_Packages_THT:TO-92_Molded_Narrow, symbol Q_NPN_EBC
- added Q? (x3): Q_NPN, TO_SOT_Packages_THT:TO-92_Molded_Narrow, symbol Q_NPN_EBC
- added R?: 1k, symbol R
- added R? (x3): 1k, Resistors_ThroughHole:Resistor_Horizontal_RM10mm, symbol R
- renumbered GND_DIST_1 to E-STOP
Connections:
- wire segments 36 -> 129
- no-connect marks 0 -> 2
Other:
- note added: "12V_IN"
- note added: "5V"
- note added: "COM"
- note added: "CR+"
- note added: "CR_1 / OVER_PRS_2"
- note added: "E-STOP COM"
- note added: "E-STOP_1 / CR-"
- note added: "E-STOP_MON"
- note added: "HI_PRESS_RLY"
- note added: "LEVEL_SW"
- note added: "OVR_PRS_1 / E-STOP_2"
- note added: "SAP_FLOW"
- note added: "SPARE_DIO"
- note added: "SPARE_RLY"
- note added: "SUMP_RLY"
- note added: "WATER_FLOW"
- note removed: "4"
- note removed: "5"
- note removed: "6"
- note removed: "7"
- note removed: "GND"
- note removed: "IGN"
- note removed: "V_BATT"
- moved on the sheet: E-STOP, U1
