File: pcb/sap-pcb.kicad_pcb (KiCad board)
At the start: 2 copper layers, 17 parts, among them P1 DROK_DC_DC_CONVERTER, Q1 Q_NPN, Q2 Q_NPN, Q3 Q_NPN, Q4 Q_NPN, U1 Arduino_Nano

Commit message: almost completed pcb design.
Parts:
- moved POWER1 104.0 mm to (90.0, 57.0), turned to 270 degrees
- moved D2 91.9 mm to (149.0, 84.0), turned to 270 degrees
- moved D3 84.1 mm to (139.0, 84.0), turned to 270 degrees
- moved CONTROL1 79.0 mm to (98.0, 117.0)
- moved R2 78.7 mm to (144.0, 99.0), turned to 90 degrees
- moved D4 78.2 mm to (129.0, 84.0), turned to 270 degrees
- moved P1 74.1 mm to (103.0, 56.0)
- moved R3 66.6 mm to (134.0, 99.0), turned to 90 degrees
- moved Q1 65.6 mm to (112.0, 105.0)
- moved D1 61.6 mm to (118.0, 84.0), turned to 270 degrees
- moved R4 53.8 mm to (124.0, 99.0), turned to 90 degrees
- moved R1 48.9 mm to (113.0, 89.0), turned to 270 degrees
- moved Q2 39.1 mm to (143.0, 105.0)
- moved U1 38.8 mm to (170.0, 76.0), turned to 270 degrees
- moved Q4 37.1 mm to (123.0, 105.0)
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Routing:
- net GND: track 0.00 -> 296.5 mm
- net Net-(D1-Pad2): track 0.00 -> 105.9 mm
- net Net-(D1-Pad1): track 0.00 -> 90.6 mm
- net Net-(R1-Pad1): track 0.00 -> 86.0 mm
- net Net-(CONTROL1-Pad14): track 0.00 -> 74.8 mm
- net Net-(R4-Pad2): track 0.00 -> 64.9 mm
- net Net-(CONTROL1-Pad15): track 0.00 -> 60.2 mm
- net Net-(CONTROL1-Pad13): track 0.00 -> 59.0 mm
- net Net-(CONTROL1-Pad12): track 0.00 -> 57.9 mm
- net Net-(R3-Pad2): track 0.00 -> 56.6 mm
- net Net-(R2-Pad2): track 0.00 -> 47.6 mm
- net Net-(CONTROL1-Pad9): track 0.00 -> 31.1 mm
- net Net-(CONTROL1-Pad10): track 0.00 -> 27.6 mm
- net Net-(CONTROL1-Pad11): track 0.00 -> 25.6 mm
- net Net-(P1-Pad1): track 0.00 -> 13.4 mm
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Other:
- board outline added: 103 x 72 mm

Commit message: finished pcb design.
Parts:
- added ?: MOUNTING_HOLE, sap-pcb:MOUNTING_HOLE, F.Cu at (88.0, 57.0)
- added ?: MOUNTING_HOLE, sap-pcb:MOUNTING_HOLE, F.Cu at (88.0, 119.0)
- added ?: MOUNTING_HOLE, sap-pcb:MOUNTING_HOLE, F.Cu at (181.0, 119.0)
- added ?: MOUNTING_HOLE, sap-pcb:MOUNTING_HOLE, F.Cu at (181.0, 57.0)
- moved POWER1 9.00 mm to (90.0, 66.0)
- moved U1 4.00 mm to (166.0, 76.0)
Routing:
- net Net-(P1-Pad1): track 13.4 -> 120.5 mm, vias 0 -> 2
- net Net-(CONTROL1-Pad3): track 0.00 -> 85.8 mm, vias 0 -> 2
- net Net-(CONTROL1-Pad1): track 5.00 -> 90.2 mm
- net Net-(CONTROL1-Pad4): track 0.00 -> 84.4 mm, vias 0 -> 2
- net GND: track 296.5 -> 312.7 mm
- net Net-(CONTROL1-Pad13): track 59.0 -> 55.1 mm
- net Net-(CONTROL1-Pad15): track 60.2 -> 56.9 mm
- net Net-(R4-Pad2): track 64.9 -> 62.8 mm
- net Net-(CONTROL1-Pad14): track 74.8 -> 72.8 mm
- net Net-(R1-Pad1): track 86.0 -> 84.5 mm
- net Net-(R2-Pad2): track 47.6 -> 46.2 mm
- net Net-(R3-Pad2): track 56.6 -> 55.6 mm
